File: BMP280Tiny/BMP280Tiny.kicad_pcb (KiCad board)
At the start: 2 copper layers, 33.1 x 49.6 mm, 26 parts, among them J1 Programming Port, U1 ATtiny88-A, U2 AMS1117-5.0, U3 BMP280, U4 AMS1117-3.3

Commit message: work on vario board
Parts:
- added C10: 0.1uF, Capacitor_SMD:C_0603_1608Metric_Pad1.08x0.95mm_HandSolder, F.Cu at (116.0, 71.5)
- added C11: 22uF 16V X5R, Capacitor_SMD:C_0805_2012Metric_Pad1.18x1.45mm_HandSolder, F.Cu at (99.7, 72.3)
- added C12: 22uF 16V X5R, Capacitor_SMD:C_0805_2012Metric_Pad1.18x1.45mm_HandSolder, F.Cu at (99.7, 75.3)
- added C13: 10nF, Capacitor_SMD:C_0603_1608Metric_Pad1.08x0.95mm_HandSolder, F.Cu at (116.0, 74.0)
- added C14: 2.2uF 50V X5R, Capacitor_SMD:C_0805_2012Metric_Pad1.18x1.45mm_HandSolder, F.Cu at (99.7, 78.3)
- added C15: 0.1uF, Capacitor_SMD:C_0603_1608Metric_Pad1.08x0.95mm_HandSolder, F.Cu at (116.0, 76.5)
- added C16: 22uF 16V X5R, Capacitor_SMD:C_0805_2012Metric_Pad1.18x1.45mm_HandSolder, F.Cu at (99.7, 81.3)
- added C17: 22uF 16V X5R, Capacitor_SMD:C_0805_2012Metric_Pad1.18x1.45mm_HandSolder, F.Cu at (99.7, 84.3)
- added C8: 10nF, Capacitor_SMD:C_0603_1608Metric_Pad1.08x0.95mm_HandSolder, F.Cu at (116.0, 69.0)
- added C9: 2.2uF 50V X5R, Capacitor_SMD:C_0805_2012Metric_Pad1.18x1.45mm_HandSolder, F.Cu at (99.7, 69.3)
- added L1: 6.8uH, Library:L_Abracon_ASPI-0310FS, F.Cu at (120.7, 70.1)
- added L2: 5.6uH, Library:L_Abracon_ASPI-0310FS, F.Cu at (120.7, 74.7)
- added R10: 100k, Resistor_SMD:R_0603_1608Metric_Pad0.98x0.95mm_HandSolder, F.Cu at (116.0, 81.6)
- added R11: 22.1k, Resistor_SMD:R_0805_2012Metric_Pad1.20x1.40mm_HandSolder, F.Cu at (104.5, 88.8)
- added R8: 100k, Resistor_SMD:R_0603_1608Metric_Pad0.98x0.95mm_HandSolder, F.Cu at (116.0, 79.0)
- added R9: 13.7k, Resistor_SMD:R_0805_2012Metric_Pad1.20x1.40mm_HandSolder, F.Cu at (104.5, 85.9)
- added SW1: SW_DPST_x2, Library:SW_19x12, F.Cu at (124.5, 95.9)
- added U5: LMR51430, Package_TO_SOT_SMD:SOT-23-6_Handsoldering, F.Cu at (116.7, 85.3)
- added U6: LMR51430, Package_TO_SOT_SMD:SOT-23-6_Handsoldering, F.Cu at (116.7, 90.0)
- moved G*** 31.3 mm to (176.0, 91.4)
- moved C3 3.42 mm to (161.9, 96.5)
- moved H4 3.42 mm to (159.4, 113.6)
- moved R1 3.42 mm to (154.9, 88.4)
- moved R3 3.42 mm to (162.6, 101.1)
- moved U1 3.42 mm to (155.3, 97.0)
- moved D2 3.42 mm to (147.7, 112.8)
- moved R2 3.42 mm to (153.1, 106.1)
- moved C2 3.42 mm to (148.5, 97.1)
- moved D1 3.42 mm to (162.6, 103.2)
- moved H3 3.42 mm to (156.1, 113.7)
Connections:
- C6 pad 2: Net-(U3-VDD) -> 3.3V
- H1 pad 1: Net-(U2-VI) -> VIN
- R4 pad 2: Net-(U3-VDD) -> 3.3V
- R5 pad 2: Net-(U3-VDD) -> 3.3V
- R6 pad 2: Net-(U3-VDD) -> 3.3V
- U3 pad 6: Net-(U3-VDD) -> 3.3V
- U3 pad 8: Net-(U3-VDD) -> 3.3V
Routing:
- net Net-(J1-Pin_3): track 34.8 -> 3.44 mm
- net Net-(J1-Pin_5): track 15.9 -> 5.57 mm, vias 1 -> 0
- net 5V: track 45.4 -> 35.1 mm
- net Net-(U1-SCL/PC5): track 29.8 -> 25.0 mm, vias 2 -> 1
- net GND: track 70.8 -> 66.8 mm, vias 16 -> 14
- net Net-(U1-SDA/PC4): track 29.2 -> 25.9 mm, vias 2 -> 1
- removed copper zone on F.Cu, net 5V
Other:
- board size 33.1 x 49.6 mm -> 47.9 x 49.6 mm
